Commit message: Moveit configured, commands are working, visual modifications

File: src/robotic_4dof_arm/urdf/arm.urdf.xacro (robot description, xacro)
@@ -69,6 +69,6 @@
       <cylinder radius="${arm_base_link_radius}" length="${arm_base_link_height}"/>
     </geometry>
-    <material name="orange">
-      <color rgba="0.85 0.035 0 1"/>
+    <material name="black">
+      <color rgba="0.1 0.1 0.1 1"/>
     </material>
   </visual>
@@ -85,5 +85,5 @@
     <parent link="world"/>
     <child link="arm_base_link"/>
-    <origin xyz="0.0 0 ${d1}" rpy="0 0 0"/>
+    <origin xyz="0.0 0 0.01" rpy="0 0 0"/>
     <limit lower="-3.14" upper="3.14" effort="150" velocity="3.14"/>
     <axis xyz="0 0 1"/>
@@ -97,6 +97,6 @@
         <cylinder radius="0.025" length="${a2}"/>
       </geometry>
-      <material name="blue">
-        <color rgba="0.035 0.035 0.85 1"/>
+      <material name="pale_blue">
+        <color rgba="0.6 0.8 1.0 1"/>
       </material>
     </visual>
@@ -118,22 +118,46 @@
     <axis xyz="0 1 0"/>
   </joint>
+  <!-- ==================== BASE-UPPER ARM (cosmetic joint) ==================== -->
+  <link name="base_upper_link">
+    <visual>
+      <origin xyz="0 0 0" rpy="1.5707 0 0"/>
+      <geometry>
+        <cylinder radius="0.0375" length="0.06"/>
+      </geometry>
+      <material name="black">
+        <color rgba="0.1 0.1 0.1 1"/>
+      </material>
+    </visual>
+    <collision>
+      <origin xyz="0 0 0" rpy="1.5707 0 0"/>
+      <geometry>
+        <cylinder radius="0.025" length="0.06"/>
+      </geometry>
+    </collision>
+    <xacro:cylinder_inertia m="0.3" r="0.025" h="0.06"/>
+  </link>
+  <joint name="base_upper_joint" type="fixed">
+    <parent link="arm_base_link"/>
+    <child link="base_upper_link"/>
+    <origin xyz="0 0 0.01" rpy="0 -1.5707 0"/>
+  </joint>
   <!-- ==================== UPPER-FORE ARM (elbow sphere) ==================== -->
   <link name="upper_forearm_link">
     <visual>
-      <origin xyz="0 0 0" rpy="0 0 0"/>
-      <geometry>
-        <sphere radius="0.0375"/>
-      </geometry>
-      <material name="cyan">
-        <color rgba="0.035 0.85 0.85 1"/>
-      </material>
-    </visual>
-    <collision>
-      <origin xyz="0 0 0" rpy="0 0 0"/>
-      <geometry>
-        <sphere radius="0.025"/>
-      </geometry>
-    </collision>
-    <xacro:sphere_inertia m="0.3" r="0.025"/>
+      <origin xyz="0 0 0" rpy="1.5707 0 0"/>
+      <geometry>
+        <cylinder radius="0.0375" length="0.06"/>
+      </geometry>
+      <material name="black">
+        <color rgba="0.1 0.1 0.1 1"/>
+      </material>
+    </visual>
+    <collision>
+      <origin xyz="0 0 0" rpy="1.5707 0 0"/>
+      <geometry>
+        <cylinder radius="0.025" length="0.06"/>
+      </geometry>
+    </collision>
+    <xacro:cylinder_inertia m="0.3" r="0.025" h="0.06"/>
   </link>
   <!-- Fixed cosmetic elbow sphere at end of upper arm -->
@@ -151,6 +175,6 @@
         <cylinder radius="0.022" length="${a3}"/>
       </geometry>
-      <material name="green">
-        <color rgba="0.035 0.85 0.035 1"/>
+      <material name="pale_blue">
+        <color rgba="0.6 0.8 1.0 1"/>
       </material>
     </visual>
@@ -174,19 +198,19 @@
   <link name="forearm_wrist_link">
     <visual>
-      <origin xyz="0 0 0" rpy="0 0 0"/>
-      <geometry>
-        <sphere radius="0.0375"/>
-      </geometry>
-      <material name="cyan">
-        <color rgba="0.035 0.85 0.85 1"/>
-      </material>
-    </visual>
-    <collision>
-      <origin xyz="0 0 0" rpy="0 0 0"/>
-      <geometry>
-        <sphere radius="0.025"/>
-      </geometry>
-    </collision>
-    <xacro:sphere_inertia m="0.3" r="0.025"/>
+      <origin xyz="0 0 0" rpy="1.5707 0 0"/>
+      <geometry>
+        <cylinder radius="0.0375" length="0.06"/>
+      </geometry>
+      <material name="black">
+        <color rgba="0.1 0.1 0.1 1"/>
+      </material>
+    </visual>
+    <collision>
+      <origin xyz="0 0 0" rpy="1.5707 0 0"/>
+      <geometry>
+        <cylinder radius="0.025" length="0.06"/>
+      </geometry>
+    </collision>
+    <xacro:cylinder_inertia m="0.3" r="0.025" h="0.06"/>
   </link>
   <!-- Fixed cosmetic wrist sphere at end of forearm -->
@@ -204,6 +228,6 @@
         <cylinder radius="0.02" length="${d4}"/>
       </geometry>
-      <material name="red">
-        <color rgba="0.85 0.035 0.035 1"/>
+      <material name="pale_blue">
+        <color rgba="0.6 0.8 1.0 1"/>
       </material>
     </visual>
@@ -232,6 +256,6 @@
         <cylinder radius="0.018" length="${d5}"/>
       </geometry>
-      <material name="cyan">
-        <color rgba="0.035 0.85 0.85 1"/>
+      <material name="pale_blue">
+        <color rgba="0.6 0.8 1.0 1"/>
       </material>
     </visual>
@@ -252,4 +276,28 @@
     <axis xyz="0 0 1"/>
   </joint>
+  <!-- ==================== WRIST-GRIPPER (cosmetic joint) ==================== -->
+  <link name="wrist_gripper_link">
+    <visual>
+      <origin xyz="0 0 0" rpy="0 0 0"/>
+      <geometry>
+        <cylinder radius="0.025" length="0.04"/>
+      </geometry>
+      <material name="black">
+        <color rgba="0.1 0.1 0.1 1"/>
+      </material>
+    </visual>
+    <collision>
+      <origin xyz="0 0 0" rpy="0 0 0"/>
+      <geometry>
+        <cylinder radius="0.02" length="0.04"/>
+      </geometry>
+    </collision>
+    <xacro:cylinder_inertia m="0.1" r="0.02" h="0.04"/>
+  </link>
+  <joint name="wrist_gripper_joint" type="fixed">
+    <parent link="wrist_link"/>
+    <child link="wrist_gripper_link"/>
+    <origin xyz="0 0 ${d4}" rpy="-1.5707 0 0"/>
+  </joint>
   <!-- ==================== GRIPPER BASE LINK (tool flange / wrist-3) ==================== -->
   <!-- d6 = 0.082 m -->
@@ -260,6 +308,6 @@
         <box size="0.008 0.04 0.04"/>
       </geometry>
-      <material name="cyan">
-        <color rgba="0.035 0.85 0.85 1"/>
+      <material name="black">
+        <color rgba="0.1 0.1 0.1 1"/>
       </material>
     </visual>
@@ -288,6 +336,6 @@
         <box size="0.02 0.005 0.1"/>
       </geometry>
-      <material name="cyan">
-        <color rgba="0.035 0.85 0.85 1"/>
+      <material name="pale_blue">
+        <color rgba="0.6 0.8 1.0 1"/>
       </material>
     </visual>
@@ -314,6 +362,6 @@
         <box size="0.02 0.005 0.1"/>
       </geometry>
-      <material name="cyan">
-        <color rgba="0.035 0.85 0.85 1"/>
+      <material name="pale_blue">
+        <color rgba="0.6 0.8 1.0 1"/>
       </material>
     </visual>
@@ -346,15 +394,21 @@
   <joint name="upper_arm_joint">
     <command_interface name="position"/>
-    <state_interface name="position"/>
+    <state_interface name="position">
+      <param name="initial_value">1.57</param>
+    </state_interface>
     <state_interface name="velocity"/>
   </joint>
   <joint name="forearm_joint">
     <command_interface name="position"/>
-    <state_interface name="position"/>
+    <state_interface name="position">
+      <param name="initial_value">-1.57</param>
+    </state_interface>
     <state_interface name="velocity"/>
   </joint>
   <joint name="wrist_joint">
     <command_interface name="position"/>
-    <state_interface name="position"/>
+    <state_interface name="position">
+      <param name="initial_value">-1.57</param>
+    </state_interface>
     <state_interface name="velocity"/>
   </joint>

Commit message: Added a scene manager for moveit

File: src/robotic_4dof_arm/urdf/arm.urdf.xacro (robot description, xacro)
@@ -381,4 +381,11 @@
     <axis xyz="0 1 0"/>
   </joint>
+  <!-- ==================== GRIPPER TCP (tool center point) ==================== -->
+  <link name="gripper_tcp"/>
+  <joint name="gripper_base_to_tcp" type="fixed">
+    <parent link="gripper_base_link"/>
+    <child link="gripper_tcp"/>
+    <origin xyz="0.0 0.0 0.075" rpy="0.0 0.0 0.0"/>
+  </joint>
   <!-- =================================================== -->
   <!-- ros2_control hardware interface -->

Commit message: The arm is working and completing its whole routine perfectly

File: src/robotic_4dof_arm/urdf/arm.urdf.xacro (robot description, xacro)
@@ -129,10 +129,4 @@
       </material>
     </visual>
-    <collision>
-      <origin xyz="0 0 0" rpy="1.5707 0 0"/>
-      <geometry>
-        <cylinder radius="0.025" length="0.06"/>
-      </geometry>
-    </collision>
     <xacro:cylinder_inertia m="0.3" r="0.025" h="0.06"/>
   </link>
@@ -153,10 +147,4 @@
       </material>
     </visual>
-    <collision>
-      <origin xyz="0 0 0" rpy="1.5707 0 0"/>
-      <geometry>
-        <cylinder radius="0.025" length="0.06"/>
-      </geometry>
-    </collision>
     <xacro:cylinder_inertia m="0.3" r="0.025" h="0.06"/>
   </link>
@@ -206,10 +194,4 @@
       </material>
     </visual>
-    <collision>
-      <origin xyz="0 0 0" rpy="1.5707 0 0"/>
-      <geometry>
-        <cylinder radius="0.025" length="0.06"/>
-      </geometry>
-    </collision>
     <xacro:cylinder_inertia m="0.3" r="0.025" h="0.06"/>
   </link>
@@ -287,10 +269,4 @@
       </material>
     </visual>
-    <collision>
-      <origin xyz="0 0 0" rpy="0 0 0"/>
-      <geometry>
-        <cylinder radius="0.02" length="0.04"/>
-      </geometry>
-    </collision>
     <xacro:cylinder_inertia m="0.1" r="0.02" h="0.04"/>
   </link>

Commit message: fixed edge detection and object detection, added contact points to the grippers

File: src/robotic_4dof_arm/urdf/arm.urdf.xacro (robot description, xacro)
@@ -316,5 +316,5 @@
       </material>
     </visual>
-    <collision>
+    <collision name="right_prong_link_collision">
       <origin xyz="0 0 0.018" rpy="0 0 0"/>
       <geometry>
@@ -328,5 +328,5 @@
     <child link="right_prong_link"/>
     <origin xyz="0 0.02 0.018" rpy="0 0 0"/>
-    <limit lower="0" upper="0.08" effort="10" velocity="1.0"/>
+    <limit lower="-0.08" upper="0.08" effort="10" velocity="1.0"/>
     <axis xyz="0 1 0"/>
   </joint>
@@ -342,5 +342,5 @@
       </material>
     </visual>
-    <collision>
+    <collision name="left_prong_link_collision">
       <origin xyz="0 0 0.018" rpy="0 0 0"/>
       <geometry>
@@ -354,5 +354,5 @@
     <child link="left_prong_link"/>
     <origin xyz="0 -0.02 0.018" rpy="0 0 0"/>
-    <limit lower="-0.08" upper="0" effort="10" velocity="1.0"/>
+    <limit lower="-0.08" upper="0.08" effort="10" velocity="1.0"/>
     <axis xyz="0 1 0"/>
   </joint>
@@ -425,4 +425,12 @@
     <minDepth>0.001</minDepth>
     <maxVel>0.1</maxVel>
+    <sensor name="right_prong_contact" type="contact">
+      <always_on>true</always_on>
+      <update_rate>50</update_rate>
+      <contact>
+        <collision>right_prong_link_collision</collision>
+      </contact>
+      <topic>right_prong_contact</topic>
+    </sensor>
   </gazebo>
   <gazebo reference="left_prong_link">
@@ -433,4 +441,12 @@
     <minDepth>0.001</minDepth>
     <maxVel>0.1</maxVel>
+    <sensor name="left_prong_contact" type="contact">
+      <always_on>true</always_on>
+      <update_rate>50</update_rate>
+      <contact>
+        <collision>left_prong_link_collision</collision>
+      </contact>
+      <topic>left_prong_contact</topic>
+    </sensor>
   </gazebo>
 <!-- gz_ros2_control plugin -->
